File: HeschDevBoard/HeschDevBoard/Schematics/197504_Kalibrierumschaltbaugruppe_seriell_2017_09_06_komplett.brd (EAGLE design)
At the start: 258 parts, among them IC1 LM317BD2T, IC10 TPD2E001DRSR, IC2 EPSON RTC8564JE, IC3 ULN2003AD, IC4 ULN2003AD, IC7 MCP23017T-E/ML, IC8 MEGA32-A, IC9 045194 CP2102SMD, K1 # 035004 / TQ2SA-3V-Z TQ2SA-3V, K2 # 035004 / TQ2SA-3V-Z TQ2SA-3V, K3 # 035004 / TQ2SA-3V-Z TQ2SA-3V, K4 # 035004 / TQ2SA-3V-Z TQ2SA-3V, K5 # 035004 / TQ2SA-3V-Z TQ2SA-3V, K6 # 035004 / TQ2SA-3V-Z TQ2SA-3V, K7 # 035004 / TQ2SA-3V-Z TQ2SA-3V, K8 # 035004 / TQ2SA-3V-Z TQ2SA-3V, SW1 088037 DTSM6, SW2 088037 DTSM6, SW3 088037 DTSM6, SW4 088037 DTSM6, SW5 088037 DTSM6, U2 MC33063AD, X1 MSTB 2,5/6-GF-5,08 AU ( Phoen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, X2 MSTB 2,5/6-GF-5,08 AU ( Phoen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, X3 MSTB 2,5/6-GF-5,08 AU ( Phoen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

Commit message: 
Parts:
- added R76: 100k, rcl:R0603
- added SJ4_2: Lötjumper, jumper:SJ
- 7_SEG_KONT_1, 7_SEG_KONT_2, 7_SEG_KONT_3, 7_SEG_KONT_4: device Siebensegment_Displays:SIEBEN_SEGMENT_KONTUR_SINGLE_dig -> Siebensegment_Displays:SIEBEN_SEGMENT_KONTUR_SINGLE_DIGIT
- R4: value 100k -> 10k
- SW1, SW2, SW3, SW4, SW5: device Taster - DIcrcBeginnPtrONICS_DTSM6:DTSM6 -> Taster - DIPTRONICS_DTSM6:DTSM6
- moved DRILEGEND 31.3 mm to (0.00, -13.0)
- moved C16 13.6 mm to (111.0, 45.5), turned to 0 degrees
- moved R1 12.6 mm to (98.0, 46.5), turned to 90 degrees
- moved D7 4.50 mm to (14.5, 53.0)
- moved D8 4.50 mm to (14.5, 48.5)
- moved C20 4.00 mm to (98.8, 63.8), turned to 90 degrees
- moved D6 2.50 mm to (100.2, 56.2)
- moved C19 1.41 mm to (99.5, 60.8), turned to 180 degrees
- renumbered SJ3 to SJ4_3, SJ4 to SJ4_1
Connections:
- net AV_ledCh1 renamed AV_CHANNEL1
- net AV_ledCh2 renamed AV_CHANNEL2
- net AV_ledCh3 renamed AV_CHANNEL3
- net AV_ledCh4 renamed AV_CHANNEL4
- net DRIVE_dig_1 renamed DRIVE_DIGIT_1
- net DRIVE_dig_2 renamed DRIVE_DIGIT_2
- net DRIVE_dig_3 renamed DRIVE_DIGIT_3
- net DRIVE_dig_4 renamed DRIVE_DIGIT_4
- net KEY_BstartUpDevice_GPA0 renamed KEY_BLOCK_GPA0
- net KEY_BstartUpDevice_GPA1 renamed KEY_BLOCK_GPA1
- net KEY_BstartUpDevice_GPA2 renamed KEY_BLOCK_GPA2
- net KEY_BstartUpDevice_GPA3 renamed KEY_BLOCK_GPA3
- net SERIAL_CstartUpDevice(SCL) renamed SERIAL_CLOCK(SCL)
- net encoder_A renamed ENCODER_A
- net encoder_B renamed ENCODER_B
- new net N$23: R4.2, SJ4_2.2
- net +3V3: now also R1.2, SJ4_2.1
- net CP2102_RXD: now also SJ9.2; no longer SJ10.2
- net CP2102_TXD: now also SJ10.2; no longer SJ9.2
- net GND: now also R76.1
- net N$12: now also R76.2
- net SUPPLY_RTC: no longer R1.2, R4.2
Routing:
- net N$23: track 0.00 -> 6.01 mm
- net CP2102_TXD: track 139.2 -> 144.0 mm
- net CP2102_RXD: track 144.0 -> 140.9 mm, vias 3 -> 2
- net +3V3: track 788.0 -> 785.1 mm
- net RTC8564_INT: track 22.7 -> 24.1 mm, vias 2 -> 3
- net ENCODER_A: track 135.4 -> 136.8 mm
- net N$12: track 4.33 -> 5.69 mm
- net SUPPLY_RTC: track 27.0 -> 25.9 mm
- net GND: vias 203 -> 195
Other:
- board text added: "ENCODER"
- board text added: "Gz 2017/09/05"
- board text added: "RELAIS_BLOCK_1"
- board text added: "RELAIS_BLOCK_2"
- board text removed: "01-16"
- board text removed: "01-20"
- board text removed: "Gz 2017/04/18"
- board text removed: "LAYER-STACK"
- board text removed: "RELAIS_BstartUpDevice_1"
- board text removed: "RELAIS_BstartUpDevice_2"
- board text removed: "encoder"
