File: HeschDevBoard/HeschDevBoard/Schematics/197504_Kalibrierumschaltbaugruppe_seriell_2017_09_06_komplett.sch (EAGLE design)
At the start: 247 parts, among them IC1 LM317BD2T, IC10 TPD2E001DRSR, IC2 EPSON RTC8564JE, IC3 ULN2003AD, IC4 ULN2003AD, IC7 MCP23017T-E/ML, IC8 MEGA32-A, IC9 045194 CP2102SMD, K1 # 035004 / TQ2SA-3V-Z TQ2SA-3V, K2 # 035004 / TQ2SA-3V-Z TQ2SA-3V, K3 # 035004 / TQ2SA-3V-Z TQ2SA-3V, K4 # 035004 / TQ2SA-3V-Z TQ2SA-3V, K5 # 035004 / TQ2SA-3V-Z TQ2SA-3V, K6 # 035004 / TQ2SA-3V-Z TQ2SA-3V, K7 # 035004 / TQ2SA-3V-Z TQ2SA-3V, K8 # 035004 / TQ2SA-3V-Z TQ2SA-3V, SW1 088037 DTSM6, SW2 088037 DTSM6, SW3 088037 DTSM6, SW4 088037 DTSM6, SW5 088037 DTSM6, U2 MC33063AD, X1 MSTB 2,5/6-GF-5,08 AU ( Phoen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, X2 MSTB 2,5/6-GF-5,08 AU ( Phoen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, X3 MSTB 2,5/6-GF-5,08 AU ( Phoen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

Commit message: 
Parts:
- removed SJ3, SJ4: Lötjumper, jumper:SJ
- added R76: 100k, rcl:R-EU_R0603
- added SJ4_1, SJ4_2, SJ4_3: Lötjumper, jumper:SJ
- R4: value 100k -> 10k
- SW1, SW2, SW3, SW4, SW5: device Taster - DIcrcBeginnPtrONICS_DTSM6:DIP_DTSM6SMD -> Taster - DIPTRONICS_DTSM6:DIP_DTSM6SMD
Connections:
- net AV_ledCh1 renamed AV_CHANNEL1
- net AV_ledCh2 renamed AV_CHANNEL2
- net AV_ledCh3 renamed AV_CHANNEL3
- net AV_ledCh4 renamed AV_CHANNEL4
- net DRIVE_dig_1 renamed DRIVE_DIGIT_1
- net DRIVE_dig_2 renamed DRIVE_DIGIT_2
- net DRIVE_dig_3 renamed DRIVE_DIGIT_3
- net DRIVE_dig_4 renamed DRIVE_DIGIT_4
- net KEY_BstartUpDevice_GPA0 renamed KEY_BLOCK_GPA0
- net KEY_BstartUpDevice_GPA1 renamed KEY_BLOCK_GPA1
- net KEY_BstartUpDevice_GPA2 renamed KEY_BLOCK_GPA2
- net KEY_BstartUpDevice_GPA3 renamed KEY_BLOCK_GPA3
- net SERIAL_CstartUpDevice(SCL) renamed SERIAL_CLOCK(SCL)
- net encoder_A renamed ENCODER_A
- net encoder_B renamed ENCODER_B
- new net N$23: R4.2, SJ4_2.2
- net +3V3: now also R1.2, SJ4_2.1
- net CLKOUT: now also SJ4_1.2; no longer SJ4.2
- net CLK_OUT_LED: now also SJ4_1.1; no longer SJ4.1
- net CP2102_RXD: now also SJ9.2; no longer SJ10.2
- net CP2102_TXD: now also SJ10.2; no longer SJ9.2
- net GND: now also R76.1
- net N$12: now also R76.2
- net RTC8564_INT: now also SJ4_3.2; no longer SJ3.2
- net RTC_INT_LED: now also SJ4_3.1; no longer SJ3.1
- net SUPPLY_RTC: no longer R1.2, R4.2
Other:
- note added: "Encoders"
- note added: "Neue Lib Displays.lbr im Standard-Pfad !"
- note added: "Real Time Clock"
- note added: "ToDo-Liste"
- note added: "erl. Gz 2017_09_05"
- note removed: "Real Time CstartUpDevice"
- note removed: "encoders"
